File: regulator_pcb.kicad_sch (KiCad schematic)
At the start: 0 parts

Commit message: test1
Parts:
- added J1: Conn_01x08, symbol Connector_Generic:Conn_01x08
Changed lines of the file:
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@@
 	(generator_version "10.0")
 	(paper "A4")
+	(symbol
+		(lib_id "Connector_Generic:Conn_01x08")
+		(at 91.44 87.63 0)
+		(unit 1)
+		(body_style 1)
+		(exclude_from_sim no)
+		(in_bom yes)
+		(on_board yes)
+		(in_pos_files yes)
+		(dnp no)
+		(fields_autoplaced yes)
+		(property "Reference" "J1"
+			(at 93.98 87.6299 0)
+			(show_name no)
+			(do_not_autoplace no)
+			(effects
+				(font
+					(size 1.27 1.27)
+				)
+				(justify left)
+			)
+		)
+		(property "Value" "Conn_01x08"
+			(at 93.98 90.1699 0)
+			(show_name no)
+			(do_not_autoplace no)
+			(effects
+				(font
+					(size 1.27 1.27)
+				)
+				(justify left)
+			)
+		)
+		(property "Footprint" ""
+			(at 91.44 87.63 0)
+			(hide yes)
+			(show_name no)
+			(do_not_autoplace no)
+			(effects
+				(font
+					(size 1.27 1.27)
+				)
+			)
+		)
+		(property "Datasheet" ""
+			(at 91.44 87.63 0)
+			(hide yes)
+			(show_name no)
+			(do_not_autoplace no)
+			(effects
+				(font
+					(size 1.27 1.27)
+				)
+			)
+		)
+		(property "Description" "Generic connector, single row, 01x08, script generated (kicad-library-utils/schlib/autogen/connector/)"
+			(at 91.44 87.63 0)
+			(hide yes)
+			(show_name no)
+			(do_not_autoplace no)
+			(effects
+				(font
+					(size 1.27 1.27)
+				)
+			)
+		)
+		(pin "2"
+		)
+		(pin "7"
+		)
+		(pin "1"
+		)
+		(pin "3"
+		)
+		(pin "6"
+		)
+		(pin "5"
+		)
+		(pin "4"
+		)
+		(pin "8"
+		)
+		(instances
+			(project "regulator_pcb"
+				(path "/2cc05e58-6e83-480c-9942-7989a7c9c21f"
+					(reference "J1")
+					(unit 1)
+				)
+			)
+		)
+	)
 	(sheet_instances
 		(path "/"

Commit message: finished schematic, almost done with pcb
Parts:
- removed J1: Conn_01x08, symbol Connector_Generic:Conn_01x08
- added C1: 0.1uF, Capacitor_SMD:C_0805_2012Metric, symbol Device:C
- added C2: 2.2uF, Capacitor_SMD:C_0805_2012Metric, symbol Device:C
- added C3: 0.01uF, Capacitor_SMD:C_0805_2012Metric, symbol Device:C
- added D1: LED-RED, LED_SMD:LED_0805_2012Metric, symbol Device:LED
- added D2: LED-GREEN, LED_SMD:LED_0805_2012Metric, symbol Device:LED
- added J1, J2: Conn_01x02, Connector_PinHeader_2.54mm:PinHeader_1x02_P2.54mm_Vertical, symbol Connector_Generic:Conn_01x02
- added R1: 649, Resistor_SMD:R_0805_2012Metric, symbol Device:R
- added R2: 280, Resistor_SMD:R_0805_2012Metric, symbol Device:R
- added U1: TPS79333-EP, Package_TO_SOT_SMD:SOT-23-5, symbol Regulator_Linear:TPS79333-EP
Connections:
- new net: D1.2 (A), R1.2
- new net: C2.1, J2.1 (Pin_1), R2.1, U1.5 (OUT)
- new net: D2.2 (A), R2.2
- new net: C1.1, J1.1 (Pin_1), R1.1, U1.1 (IN), U1.3 (EN)
- new net: C3.1, U1.4 (BP)
- new net GND: C1.2, C2.2, C3.2, D1.1 (K), D2.1 (K), J1.2 (Pin_2), J2.2 (Pin_2), U1.2 (GND)
Other:
- note added: "R1 = 650 Ohm"
- note added: "R2 = 280 Ohm"
- note added: "essentially: input 5V into resistor R1 the D1 (red) LED will voltage drop 1.75V (because we're using APTD2012LSURCK). 5V - 1.75V = 3.25V drop across Resistor 1. thus, we use Ohm's Law to calculate this resistor, which is the voltage divided by current. R = V / I, so R1 voltage drop is R1 = 3.25V / 5mA = 650 Ohms"
- note added: "for the LEDs, go to DigiKey, filter by color: red & green supplier device package: 2012 or 0805 product status: active you end up with APTD2012LSURCK (red) and APTD2012LCGCK (green)"
- note added: "go to the tps793 data sheet to be able to find the capacitor / regulator information to understand what level capacitor u should be using"
- note added: "in "9.2 Typical Application" of the document, the capacitor shows 0.1 microfarad on the input and 2.2 microfarad on the output. 0.01 microfarad on the bypass capacitor (bypass pin)"
- note added: "just like how we did for the LEDs, also go to DigiKey for the resistors. search up "resistors 0805", select "chip resistors surface mount," and filter by - Resistance: 280 Ohms & 650 Ohms (couldn't find 650 so settled for 649) - Supplier Device Package: 0805"
- note added: "just like the red LED, we calculate this part too. we're using APTD2012LCGCK for the green LED, so: - output that hits the resistor: 3.3V - the LED voltage drop of the green LED is 1.9V Voltage drop (across R2): 3.3V - 1.9V = 1.4V according ot Ohm's Law, or R = V / I R3 = 1.4V / 5mA = 280 Ohms for this resistor"
- note added: "since we couldn't find any 650 Ohm resistors, we change R1 to 649 (the closest one we found)"
- note added: "the input voltage is 5V, and because we found the LEDs on DigiKey, we found that the voltage drop was 1.75V. (it's in the "Voltage - Forward (Vf) (Typ)" column)"
